File: SI4735.kicad_pcb (KiCad board)
At the start: 2 copper layers, 31 parts, among them J1 Conn_01x04_Male, J2 Conn_01x02_Male, J3 Conn_01x01_Male, J4 Conn_01x03_Male, J5 Conn_01x02_Male, U1 AMS1117-3.3, U2 Si4735-D60-GU, Y1 32.768kHz

Commit message: Update Project Data
Parts:
- removed C13: 20uF, Capacitor_SMD:CP_Elec_6.3x5.8
- removed J1: Conn_01x04_Male, Connector_Wago:Wago_734-134_1x04_P3.50mm_Vertical
- added C14: 20uF, Capacitor_THT:CP_Radial_D5.0mm_P2.00mm, F.Cu at (228.4, 48.6)
- added C15: 20uF, Capacitor_THT:CP_Radial_D5.0mm_P2.00mm, F.Cu at (235.1, 49.5)
- added D1: BAW75, Diode_THT:D_DO-35_SOD27_P7.62mm_Horizontal, F.Cu at (203.8, 75.6)
- added D2: BAW75, Diode_THT:D_DO-35_SOD27_P7.62mm_Horizontal, F.Cu at (206.4, 68.0)
- added D3: BAW75, Diode_THT:D_DO-35_SOD27_P7.62mm_Horizontal, F.Cu at (203.4, 46.9)
- added D4: BAW75, Diode_THT:D_DO-35_SOD27_P7.62mm_Horizontal, F.Cu at (205.9, 54.5)
- added G***: LOGO, Logo:Logo, B.Cu at (219.2, 50.1)
- added J6: Conn_01x06_Male, Connector_PinHeader_2.54mm:PinHeader_1x06_P2.54mm_Vertical, B.Cu at (234.6, 53.9)
- added R10: 4.7k, Resistor_SMD:R_1206_3216Metric, B.Cu at (209.7, 71.5)
- added R11: 4.7k, Resistor_THT:R_Axial_DIN0309_L9.0mm_D3.2mm_P12.70mm_Horizontal, F.Cu at (209.8, 67.8)
- added R12: 4.7k, Resistor_SMD:R_1206_3216Metric, B.Cu at (239.1, 59.0)
- added R13: 100R, Resistor_SMD:R_1206_3216Metric, B.Cu at (226.3, 63.8)
- added R14: 4.7k, Resistor_SMD:R_1206_3216Metric, B.Cu at (239.1, 61.3)
- added U3: AMS1117-5.0, Package_TO_SOT_SMD:SOT-223-3_TabPin2, F.Cu at (215.6, 52.4)
- C1, C2, C3: footprint Capacitor_THT:C_Disc_D5.1mm_W3.2mm_P5.00mm -> Capacitor_SMD:C_1206_3216Metric; moved to B.Cu
- C10, C9: footprint Capacitor_THT:C_Disc_D5.0mm_W2.5mm_P5.00mm -> Capacitor_THT:C_Disc_D3.4mm_W2.1mm_P2.50mm
- C11, C12: value C -> 0.01uF; footprint Capacitor_THT:C_Disc_D5.0mm_W2.5mm_P5.00mm -> Capacitor_THT:C_Disc_D3.4mm_W2.1mm_P2.50mm
- C4: footprint Capacitor_SMD:CP_Elec_6.3x5.9 -> Capacitor_THT:CP_Radial_D5.0mm_P2.00mm
- C5: footprint Capacitor_THT:C_Disc_D7.5mm_W5.0mm_P5.00mm -> Capacitor_THT:C_Disc_D3.0mm_W1.6mm_P2.50mm
- C6, C7: footprint Capacitor_THT:C_Disc_D7.5mm_W5.0mm_P5.00mm -> Capacitor_THT:C_Disc_D4.3mm_W1.9mm_P5.00mm
- C8: value 470nF -> 20uF; footprint Capacitor_THT:C_Disc_D7.5mm_W5.0mm_P5.00mm -> Capacitor_THT:CP_Radial_D5.0mm_P2.00mm
- J2: value Conn_01x02_Male -> AM_IN; footprint Connector_Wago:Wago_734-132_1x02_P3.50mm_Vertical -> Connector_Coaxial:SMA_Amphenol_901-143_Horizontal
- J3: value Conn_01x01_Male -> FM_IN; footprint Connector_PinHeader_2.54mm:PinHeader_1x01_P2.54mm_Horizontal -> Connector_Coaxial:SMA_Amphenol_901-143_Horizontal
- J4: footprint Connector_Wago:Wago_734-133_1x03_P3.50mm_Vertical -> Connector_PinHeader_2.54mm:PinHeader_1x03_P2.54mm_Vertical; moved to B.Cu
- J5: footprint Connector_Wago:Wago_734-132_1x02_P3.50mm_Vertical -> Connector_PinHeader_2.54mm:PinHeader_1x02_P2.54mm_Vertical; moved to B.Cu
- L1, L2: footprint Inductor_THT:L_Radial_D18.0mm_P10.00mm -> Inductor_THT:L_Radial_D6.0mm_P4.00mm
- R1: value 10k -> 100R; footprint Resistor_THT:R_Axial_DIN0207_L6.3mm_D2.5mm_P10.16mm_Horizontal -> Resistor_SMD:R_1206_3216Metric; moved to B.Cu
- R2, R3: value 1k -> 100R; footprint Resistor_THT:R_Axial_DIN0207_L6.3mm_D2.5mm_P10.16mm_Horizontal -> Resistor_SMD:R_1206_3216Metric; moved to B.Cu
- R4, R5: footprint Resistor_THT:R_Axial_DIN0207_L6.3mm_D2.5mm_P10.16mm_Horizontal -> Resistor_SMD:R_1206_3216Metric; moved to B.Cu
- R6: value 210R -> 10k; footprint Resistor_THT:R_Axial_DIN0207_L6.3mm_D2.5mm_P10.16mm_Horizontal -> Resistor_SMD:R_1206_3216Metric; moved to B.Cu
- R7, R8: value 1k -> 0.2k; footprint Resistor_THT:R_Axial_DIN0207_L6.3mm_D2.5mm_P10.16mm_Horizontal -> Resistor_SMD:R_1206_3216Metric; moved to B.Cu
- moved R6 146.4 mm to (239.1, 56.5), turned to 180 degrees
- moved R5 143.4 mm to (239.1, 65.8), turned to 180 degrees
- moved R1 140.6 mm to (226.3, 61.6)
- moved L2 139.8 mm to (205.7, 58.0)
- moved C5 138.0 mm to (223.4, 71.2), turned to 180 degrees
- moved R7 134.2 mm to (224.5, 73.5), turned to 180 degrees
- moved R3 133.9 mm to (226.3, 68.2)
- moved C9 132.7 mm to (230.8, 70.2), turned to -90 degrees
- moved J5 131.5 mm to (229.3, 56.5)
- moved R4 128.7 mm to (239.1, 63.5), turned to 180 degrees
- moved C4 128.3 mm to (220.8, 60.9), turned to 180 degrees
- moved C1 125.2 mm to (220.6, 62.9), turned to 180 degrees
- moved C3 122.5 mm to (213.4, 75.7), turned to -90 degrees
- moved L1 121.2 mm to (200.5, 61.4), turned to 180 degrees
- moved R2 119.8 mm to (226.3, 66.0)
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Connections:
- C1 pad 2: Net-(C1-Pad2) -> GND
- C10 pad 1: Net-(C10-Pad1) -> Net-(J4-Pin_1)
- C11 pad 1: Net-(C1-Pad2) -> GND
- C12 pad 1: Net-(C1-Pad2) -> GND
- C2 pad 2: Net-(C1-Pad2) -> GND
- C3 pad 2: Net-(C1-Pad2) -> GND
- C4 pad 1: Net-(C4-Pad1) -> Net-(J6-Pin_1)
- C4 pad 2: Net-(C1-Pad2) -> GND
- C5 pad 1: Net-(C13-Pad1) -> Net-(U2-VA)
- C6 pad 1: Net-(C6-Pad1) -> Net-(D3-A)
- C7 pad 1: Net-(C7-Pad1) -> Net-(D1-A)
- C8 pad 1: Net-(C8-Pad1) -> Net-(U2-VA)
- C8 pad 2: Net-(C8-Pad2) -> GND
- C9 pad 1: Net-(C9-Pad1) -> Net-(J4-Pin_3)
- J2 pad 1: Net-(C1-Pad2) -> Net-(D3-A)
- J2 pad 2: Net-(C8-Pad1) -> GND
- J3 pad 1: Net-(C7-Pad1) -> Net-(D1-A)
- J4 pad 1: Net-(C9-Pad1) -> Net-(J4-Pin_1)
- J4 pad 2: Net-(C1-Pad2) -> GND
- J4 pad 3: Net-(C10-Pad1) -> Net-(J4-Pin_3)
- J5 pad 1: Net-(C1-Pad2) -> GND
- J5 pad 2: Net-(C13-Pad1) -> Net-(J5-Pin_2)
- L1 pad 1: Net-(C6-Pad1) -> Net-(D1-A)
- L1 pad 2: Net-(C1-Pad2) -> Net-(D3-A)
- L2 pad 1: Net-(C8-Pad2) -> Net-(D3-A)
- L2 pad 2: Net-(C1-Pad2) -> GND
- R1 pad 2: Net-(J1-Pad1) -> Net-(J6-Pin_2)
- R2 pad 1: Net-(R2-Pad1) -> Net-(U2-SCLK)
- R2 pad 2: Net-(J1-Pad2) -> Net-(J6-Pin_4)
- R3 pad 1: Net-(R3-Pad1) -> Net-(U2-SDIO)
- R3 pad 2: Net-(J1-Pad3) -> Net-(J6-Pin_5)
- R4 pad 1: Net-(C4-Pad1) -> Net-(J6-Pin_1)
- R4 pad 2: Net-(R2-Pad1) -> Net-(J6-Pin_4)
- R5 pad 1: Net-(C4-Pad1) -> Net-(J6-Pin_1)
- R5 pad 2: Net-(R3-Pad1) -> Net-(J6-Pin_5)
- R6 pad 1: Net-(C4-Pad1) -> Net-(J6-Pin_1)
- R6 pad 2: Net-(C1-Pad2) -> Net-(J6-Pin_2)
- U1 pad 1: Net-(C1-Pad2) -> GND
- U1 pad 2: Net-(C4-Pad1) -> Net-(J6-Pin_1)
- U1 pad 3: Net-(C13-Pad1) -> Net-(J5-Pin_2)
- U2 pad 1: Net-(U2-Pad1) -> unconnected-(U2-DOUT-Pad1)
- U2 pad 10: Net-(U2-Pad10) -> unconnected-(U2-NC-Pad10)
- U2 pad 11: Net-(U2-Pad11) -> unconnected-(U2-NC-Pad11)
- U2 pad 13: Net-(C1-Pad2) -> GND
- U2 pad 14: Net-(C1-Pad2) -> GND
- U2 pad 16: Net-(C4-Pad1) -> Net-(U2-~{SEN})
- U2 pad 17: Net-(R3-Pad1) -> Net-(U2-SCLK)
- U2 pad 18: Net-(R2-Pad1) -> Net-(U2-SDIO)
- U2 pad 2: Net-(U2-Pad2) -> unconnected-(U2-DFS-Pad2)
- U2 pad 20: Net-(C13-Pad1) -> Net-(J6-Pin_1)
- U2 pad 21: Net-(C4-Pad1) -> Net-(U2-VA)
- U2 pad 6: Net-(U2-Pad6) -> unconnected-(U2-NC-Pad6)
- U2 pad 7: Net-(U2-Pad7) -> unconnected-(U2-NC-Pad7)
- U2 pad 9: Net-(C1-Pad2) -> GND
Routing:
- net GND: track 0.00 -> 6112.9 mm
- net Net-(J6-Pin_1): track 0.00 -> 171.5 mm
- net Net-(J5-Pin_2): track 0.00 -> 124.7 mm
- net Net-(D3-A): track 0.00 -> 101.2 mm
- net Net-(U2-VA): track 0.00 -> 93.8 mm
- net Net-(D1-A): track 0.00 -> 27.3 mm
- net Net-(J6-Pin_3): track 0.00 -> 25.0 mm
- net Net-(J6-Pin_5): track 0.00 -> 14.9 mm
- net Net-(J6-Pin_2): track 0.00 -> 13.4 mm
- net Net-(J6-Pin_4): track 0.00 -> 12.6 mm
- net Net-(U2-AMI): track 0.00 -> 10.2 mm
- net Net-(U2-LOUT/[DFS]): track 0.00 -> 9.26 mm
- net Net-(U2-~{RST}): track 0.00 -> 9.21 mm
- net Net-(U2-~{SEN}): track 0.00 -> 8.85 mm
- net Net-(U2-RCLK): track 0.00 -> 8.67 mm
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Other:
- board outline added: 50.8 x 38.8 mm
- net class Default removed
- board text added: "+"
- board text added: "3.3 V"
- board text added: "AM IN"
- board text added: "AMS 1117 -3.3"
- board text added: "AMS 1117 -5.0"
- board text added: "Control"
- board text added: "FM IN"
- board text added: "G"
- board text added: "GND"
- board text added: "L"
- board text added: "Power"
- board text added: "R"
- board text added: "RST"
- board text added: "SCLK/SCL"
- board text added: "SDIO/SDA"
- board text added: "SEN"
- board text added: "Si4735-based radio. Developed by A. Ivanov 14.08.2022"
